Commit message: Update apartment

File: resources/Modified_ApartmentECAI.urdf (robot description, URDF)
Before this commit: robot Apartment, 86 links, 85 joints
Links:
- removed link table
- added link SM_DiningTable, mass 36.17988967895508; collision mesh filename=file://ApartmentECAI/meshes/stl/UCX_DiningTable_001.stl scale=1.0 1.0 1.0; collision mesh filename=file://ApartmentECAI/meshes/stl/UCX_DiningTable_002.stl scale=1.0 1.0 1.0
Joints:
- removed joint table_joint
- added joint SM_DiningTable_joint: type fixed, parent Apartment, child SM_DiningTable, origin xyz=4.059035468329589 -6.57453813671817 0.37744309672918996 rpy=0.0 0.0 1.570798397064209
